Commit message: cleanup and leg urdf loading

File: leg.urdf (robot description, URDF)
Before this commit: robot vision60, 4 links, 3 joints
Links:
- link body: geometry visual box size=0.83 0.25 0.19
- link hip0: geometry visual box size=0.15 0.09 0.15
- link lower0: geometry visual cylinder length=0.3407 radius=0.02
- link upper0: geometry visual box size=0.34 0.055 0.075
Joints:
- joint body_hip: child  -> hip0; parent  -> body
- joint hip_upper: child  -> upper0; parent  -> hip0
- joint upper_lower: child  -> lower0; parent  -> upper0

Commit message: leg optimizer actually running, but not successfully

File: leg.urdf (robot description, URDF)
Before this commit: robot vision60, 4 links, 3 joints
Joints:
- added joint base_weld: type fixed, parent world, child body
- joint body_hip: type revolute -> continuous
- joint hip_upper: type revolute -> continuous
- joint upper_lower: type revolute -> continuous

Commit message: mesh and urdf updates, mass matrix works

File: leg.urdf (robot description, URDF)
Before this commit: robot vision60, 4 links, 4 joints
Links:
- link body: geometry visual mesh filename=mesh/Frame.obj scale=1 1 1
- link hip0: mass None -> 1.975; geometry visual mesh filename=mesh/Hip_Pod_Assembly.obj scale=1 1 1
- link lower0: mass None -> 0.525; geometry visual mesh filename=mesh/Lower_Leg_Assembly.obj scale=.001 .001 .001
- link upper0: mass None -> 2.525; geometry visual mesh filename=mesh/Leg_Assembly.obj scale=.001 .001 .001
Joints:
- joint body_hip: axis  -> 1 0 0
- joint hip_upper: axis  -> 0 -1 0
- joint upper_lower: axis  -> 0 1 0
