Commit message: decimated meshes

File: leg_v2.urdf (robot description, URDF)
Before this commit: robot vision60, 4 links, 4 joints
Links:
- link body: geometry collision box size=0.19 0.09 0.14; visual mesh filename=mesh/v4_frame.obj scale=1 1 1
- link hip0: geometry collision box size=0.19 0.09 0.14; visual mesh filename=mesh/v4_hip.obj scale=1 1 1
- link lower0: geometry collision cylinder length=0.3176 radius=0.02; visual mesh filename=mesh/v4_lower.obj scale=1 1 1
- link upper0: geometry collision box size=0.32 0.055 0.08; visual mesh filename=mesh/v4_upper.obj scale=1 1 1
Joints:
- joint hip_upper: origin xyz=0 0.0875 0 -> xyz=0 0.12 0 rpy=0 3.14 0

Commit message: fixed urdf and throwing traj works

File: leg_v2.urdf (robot description, URDF)
Before this commit: robot vision60, 4 links, 4 joints
Joints:
- joint body_hip: limit (none) -> lower=-0.53 upper=0.53 effort=375 velocity=8.6
- joint hip_upper: limit (none) -> lower=-6.28318530718 upper=6.28318530718 effort=87.5 velocity=30
- joint upper_lower: limit (none) -> lower=0 upper=3.14159265359 effort=87.5 velocity=30

Commit message: Obstacle generation and constraints, add toe to urdf

File: leg_v2.urdf (robot description, URDF)
Before this commit: robot vision60_leg, 4 links, 4 joints
Links:
- added link toe0; visual sphere radius=.05
Joints:
- added joint lower_toe: type fixed, parent lower0, child toe0, origin xyz=0.3176 0 0
- joint base_weld: origin (none) -> xyz=0.0 0.0 0.5

Commit message: fixed infeasible with all joints and bigger obst

File: leg_v2.urdf (robot description, URDF)
Before this commit: robot vision60_leg, 5 links, 5 joints
Links:
- link toe0: geometry visual sphere radius=.02
Joints:
- joint lower_toe: origin xyz=0.3176 0 0 -> xyz=0.3176 0 -0.01
